File: Display/Display.kicad_sch (KiCad schematic)
At the start: 9 parts, among them J1 Conn_01x60, J2 12402032E202A, J3 12402032E202A, J4 Conn_01x60

Commit message: before attempt to fix annotation
Connections:
- net GNDD: now also J1.50 (Pin_50), J1.52 (Pin_52), J1.54 (Pin_54), J1.56 (Pin_56), J1.58 (Pin_58); no longer J4.52 (Pin_52), J4.54 (Pin_54), J4.56 (Pin_56), J4.58 (Pin_58), J4.60 (Pin_60)
- net RCL: now also J4.56 (Pin_56); no longer J1.56 (Pin_56)
- net SR: now also J4.52 (Pin_52); no longer J1.50 (Pin_50)
- net SRCL: now also J4.58 (Pin_58); no longer J1.52 (Pin_52)
- net SRCR: now also J4.60 (Pin_60); no longer J1.54 (Pin_54)
- net ~{OE}: now also J4.54 (Pin_54); no longer J1.58 (Pin_58)

Commit message: cascade digits
Parts:
- renumbered J4 to J1, J3 to J2, J2 to J3, J1 to J4, S2 to S1, S3 to S2, S1 to S3
Changed lines of the file:
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@@
 		(on_board yes)
 		(dnp no)
-		(property "Reference" "S3"
+		(property "Reference" "S2"
 			(at 27.94 147.066 0)
 			(effects
@@
 			(project "Display"
 				(path "/4a3e89f9-ab44-4b68-b8a8-f6bfa5391fb1"
-					(reference "S3")
+					(reference "S2")
 					(unit 1)
 				)
@@
 		(dnp no)
 		(fields_autoplaced yes)
-		(property "Reference" "#PWR0254"
+		(property "Reference" "#PWR03"
 			(at 154.94 283.21 0)
 			(effects
@@
 			(project "Display"
 				(path "/4a3e89f9-ab44-4b68-b8a8-f6bfa5391fb1"
-					(reference "#PWR0254")
+					(reference "#PWR03")
 					(unit 1)
 				)
@@
 		(dnp no)
 		(fields_autoplaced yes)
-		(property "Reference" "J2"
+		(property "Reference" "J3"
 			(at 106.68 118.11 0)
 			(effects
@@
 			(project ""
 				(path "/4a3e89f9-ab44-4b68-b8a8-f6bfa5391fb1"
-					(reference "J2")
+					(reference "J3")
 					(unit 1)
 				)
@@
 		(on_board yes)
 		(dnp no)
-		(property "Reference" "#PWR0253"
+		(property "Reference" "#PWR02"
 			(at 63.5 203.2 0)
 			(effects
@@
 			(project "Display"
 				(path "/4a3e89f9-ab44-4b68-b8a8-f6bfa5391fb1"
-					(reference "#PWR0253")
+					(reference "#PWR02")
 					(unit 1)
 				)
@@
 		(on_board yes)
 		(dnp no)
-		(property "Reference" "S1"
+		(property "Reference" "S3"
 			(at 27.178 166.37 0)
 			(effects
@@
 			(project ""
 				(path "/4a3e89f9-ab44-4b68-b8a8-f6bfa5391fb1"
-					(reference "S1")
+					(reference "S3")
 					(unit 1)
 				)
@@
 		(dnp no)
 		(fields_autoplaced yes)
-		(property "Reference" "#FLG02"
+		(property "Reference" "#FLG01"
 			(at 49.53 239.395 0)
 			(effects
@@
 			(project "Display"
 				(path "/4a3e89f9-ab44-4b68-b8a8-f6bfa5391fb1"
-					(reference "#FLG02")
+					(reference "#FLG01")
 					(unit 1)
 				)
@@
 		(dnp no)
 		(fields_autoplaced yes)
-		(property "Reference" "J1"
+		(property "Reference" "J4"
 			(at 163.83 199.3899 0)
 			(effects
@@
 			(project "Display"
 				(path "/4a3e89f9-ab44-4b68-b8a8-f6bfa5391fb1"
-					(reference "J1")
+					(reference "J4")
 					(unit 1)
 				)
@@
 		(dnp no)
 		(fields_autoplaced yes)
-		(property "Reference" "J3"
+		(property "Reference" "J2"
 			(at 90.17 179.07 0)
 			(effects
@@
 			(project "Display"
 				(path "/4a3e89f9-ab44-4b68-b8a8-f6bfa5391fb1"
-					(reference "J3")
+					(reference "J2")
 					(unit 1)
 				)
@@
 		(on_board yes)
 		(dnp no)
-		(property "Reference" "S2"
+		(property "Reference" "S1"
 			(at 27.94 128.27 0)
 			(effects
@@
 			(project "Display"
 				(path "/4a3e89f9-ab44-4b68-b8a8-f6bfa5391fb1"
-					(reference "S2")
+					(reference "S1")
 					(unit 1)
 				)
@@
 		(dnp no)
 		(fields_autoplaced yes)
-		(property "Reference" "#FLG01"
+		(property "Reference" "#FLG02"
 			(at 59.055 223.52 0)
 			(effects
@@
 			(project ""
 				(path "/4a3e89f9-ab44-4b68-b8a8-f6bfa5391fb1"
-					(reference "#FLG01")
+					(reference "#FLG02")
 					(unit 1)
 				)
@@
 		(dnp no)
 		(fields_autoplaced yes)
-		(property "Reference" "J4"
+		(property "Reference" "J1"
 			(at 71.12 200.6599 0)
 			(effects
@@
 			(project "Display"
 				(path "/4a3e89f9-ab44-4b68-b8a8-f6bfa5391fb1"
-					(reference "J4")
+					(reference "J1")
 					(unit 1)
 				)
@@
 		(dnp no)
 		(fields_autoplaced yes)
-		(property "Reference" "#PWR0112"
+		(property "Reference" "#PWR01"
 			(at 49.53 285.75 0)
 			(effects
@@
 			(project "Display"
 				(path "/4a3e89f9-ab44-4b68-b8a8-f6bfa5391fb1"
-					(reference "#PWR0112")
+					(reference "#PWR01")
 					(unit 1)
 				)

Commit message: usb1
Connections:
- net GNDD: now also J4.1 (Pin_1), J4.10 (Pin_10), J4.11 (Pin_11), J4.12 (Pin_12), J4.2 (Pin_2), J4.3 (Pin_3), J4.4 (Pin_4), J4.5 (Pin_5), J4.6 (Pin_6), J4.7 (Pin_7), J4.8 (Pin_8), J4.9 (Pin_9); no longer J4.49 (Pin_49), J4.50 (Pin_50), J4.51 (Pin_51), J4.52 (Pin_52), J4.53 (Pin_53), J4.54 (Pin_54), J4.55 (Pin_55), J4.56 (Pin_56), J4.57 (Pin_57), J4.58 (Pin_58), J4.59 (Pin_59), J4.60 (Pin_60)
- net at J3.A1 (GND): now also J4.36 (Pin_36); no longer J4.24 (Pin_24)
- net at J3.A10 (RX2-): now also J4.27 (Pin_27); no longer J4.15 (Pin_15)
- net at J3.A11 (RX2+): now also J4.26 (Pin_26); no longer J4.14 (Pin_14)
- net at J3.A12 (GND): now also J4.25 (Pin_25); no longer J4.13 (Pin_13)
- net at J3.A2 (TX1+): now also J4.35 (Pin_35); no longer J4.23 (Pin_23)
- net at J3.A3 (TX1-): now also J4.34 (Pin_34); no longer J4.22 (Pin_22)
- net at J3.A4 (VBUS): now also J4.33 (Pin_33); no longer J4.21 (Pin_21)
- net at J3.A5 (CC1): now also J4.32 (Pin_32); no longer J4.20 (Pin_20)
- net at J3.A6 (D+): now also J4.31 (Pin_31); no longer J4.19 (Pin_19)
- net at J3.A7 (D-): now also J4.30 (Pin_30); no longer J4.18 (Pin_18)
- net at J3.A8 (SBU1): now also J4.29 (Pin_29); no longer J4.17 (Pin_17)
- net at J3.A9 (VBUS): now also J4.28 (Pin_28); no longer J4.16 (Pin_16)
- net at J3.B1 (GND): now also J4.13 (Pin_13); no longer J4.1 (Pin_1)
- net at J3.B10 (RX1-): now also J4.22 (Pin_22); no longer J4.10 (Pin_10)
- net at J3.B11 (RX1+): now also J4.23 (Pin_23); no longer J4.11 (Pin_11)
- net at J3.B12 (GND): now also J4.24 (Pin_24); no longer J4.12 (Pin_12)
- net at J3.B2 (TX2+): now also J4.14 (Pin_14); no longer J4.2 (Pin_2)
- net at J3.B3 (TX2-): now also J4.15 (Pin_15); no longer J4.3 (Pin_3)
- net at J3.B4 (VBUS): now also J4.16 (Pin_16); no longer J4.4 (Pin_4)
- net at J3.B5 (CC1): now also J4.17 (Pin_17); no longer J4.5 (Pin_5)
- net at J3.B6 (D+): now also J4.18 (Pin_18); no longer J4.6 (Pin_6)
- net at J3.B7 (D-): now also J4.19 (Pin_19); no longer J4.7 (Pin_7)
- net at J3.B8 (SBU2): now also J4.20 (Pin_20); no longer J4.8 (Pin_8)
- net at J3.B9 (VBUS): now also J4.21 (Pin_21); no longer J4.9 (Pin_9)
- net at J2.B12 (GND): now also J4.37 (Pin_37); no longer J4.25 (Pin_25)
- net at J2.B11 (RX1+): now also J4.38 (Pin_38); no longer J4.26 (Pin_26)
- net at J2.B10 (RX1-): now also J4.39 (Pin_39); no longer J4.27 (Pin_27)
- net at J2.B9 (VBUS): now also J4.40 (Pin_40); no longer J4.28 (Pin_28)
- net at J2.B8 (SBU2): now also J4.41 (Pin_41); no longer J4.29 (Pin_29)
- net at J2.B7 (D-): now also J4.42 (Pin_42); no longer J4.30 (Pin_30)
- net at J2.B6 (D+): now also J4.43 (Pin_43); no longer J4.31 (Pin_31)
- net at J2.B5 (CC1): now also J4.44 (Pin_44); no longer J4.32 (Pin_32)
- net at J2.B4 (VBUS): now also J4.45 (Pin_45); no longer J4.33 (Pin_33)
- net at J2.B3 (TX2-): now also J4.46 (Pin_46); no longer J4.34 (Pin_34)
- net at J2.B2 (TX2+): now also J4.47 (Pin_47); no longer J4.35 (Pin_35)
- net at J2.B1 (GND): now also J4.48 (Pin_48); no longer J4.36 (Pin_36)
- net at J2.A1 (GND): now also J4.49 (Pin_49); no longer J4.37 (Pin_37)
- net at J2.A2 (TX1+): now also J4.50 (Pin_50); no longer J4.38 (Pin_38)
- net at J2.A3 (TX1-): now also J4.51 (Pin_51); no longer J4.39 (Pin_39)
- net at J2.A4 (VBUS): now also J4.52 (Pin_52); no longer J4.40 (Pin_40)
- net at J2.A5 (CC1): now also J4.53 (Pin_53); no longer J4.41 (Pin_41)
- net at J2.A6 (D+): now also J4.54 (Pin_54); no longer J4.42 (Pin_42)
- net at J2.A7 (D-): now also J4.55 (Pin_55); no longer J4.43 (Pin_43)
- net at J2.A8 (SBU1): now also J4.56 (Pin_56); no longer J4.44 (Pin_44)
- net at J2.A9 (VBUS): now also J4.57 (Pin_57); no longer J4.45 (Pin_45)
- net at J2.A10 (RX2-): now also J4.58 (Pin_58); no longer J4.46 (Pin_46)
- net at J2.A11 (RX2+): now also J4.59 (Pin_59); no longer J4.47 (Pin_47)
- net at J2.A12 (GND): now also J4.60 (Pin_60); no longer J4.48 (Pin_48)
Other:
- moved on the sheet: J2, J3, J4

Commit message: quick save
Parts:
- removed J4: Conn_01x60, External_Parts:CON_2004850460_MOL, symbol Connector_Generic:Conn_01x60
Connections:
- net GNDD: now also J1.36 (Pin_36), J1.38 (Pin_38), J1.40 (Pin_40), J1.42 (Pin_42), J1.44 (Pin_44), J1.58 (Pin_58), J2.A1 (GND), J2.A12 (GND), J2.B1 (GND), J2.B12 (GND), J3.A1 (GND), J3.A12 (GND), J3.B1 (GND), J3.B12 (GND); no longer J1.48 (Pin_48), J1.49 (Pin_49), J1.51 (Pin_51), J1.53 (Pin_53), J1.57 (Pin_57), J1.59 (Pin_59)
- net RCL: now also J1.41 (Pin_41); no longer J1.56 (Pin_56)
- net SR: now also J1.37 (Pin_37); no longer J1.52 (Pin_52)
- net SRCL: now also J1.43 (Pin_43); no longer J1.58 (Pin_58)
- net SRCR: now also J1.45 (Pin_45); no longer J1.60 (Pin_60)
- net VCC: no longer J1.36 (Pin_36), J1.37 (Pin_37), J1.38 (Pin_38), J1.39 (Pin_39), J1.40 (Pin_40), J1.41 (Pin_41), J1.42 (Pin_42), J1.43 (Pin_43), J1.44 (Pin_44), J1.45 (Pin_45)
- net ~{OE}: now also J1.39 (Pin_39); no longer J1.54 (Pin_54)
- net CHARGER_VBUS: now reaches J3.A4 (VBUS)
- net CHARGER_VBUS: now also J1.52 (Pin_52), J3.A9 (VBUS), J3.B4 (VBUS), J3.B9 (VBUS)
- net CHARGER_CC1: now reaches J3.A5 (CC1)
- net CHARGER_CC1: now also J1.53 (Pin_53)
- net CHARGER_D+: now reaches J3.A6 (D+)
- net CHARGER_D+: now also J1.49 (Pin_49), J3.B6 (D+)
- net CHARGER_D-: now reaches J3.A7 (D-)
- net CHARGER_D-: now also J1.48 (Pin_48), J3.B7 (D-)
- net CHARGER_CC2: now reaches J3.B5 (CC1)
- net CHARGER_CC2: now also J1.51 (Pin_51)
- net DAC_VBUS: now reaches J2.B9 (VBUS)
- net DAC_VBUS: now also J1.59 (Pin_59), J2.A4 (VBUS), J2.A9 (VBUS), J2.B4 (VBUS)
- net DAC_D-: now reaches J2.B7 (D-)
- net DAC_D-: now also J1.57 (Pin_57), J2.A7 (D-)
- net DAC_D+: now reaches J2.B6 (D+)
- net DAC_D+: now also J1.56 (Pin_56), J2.A6 (D+)
- net DAC_CC2: now reaches J2.B5 (CC1)
- net DAC_CC2: now also J1.54 (Pin_54)
- net DAC_CC1: now reaches J2.A5 (CC1)
- net DAC_CC1: now also J1.60 (Pin_60)
- no-connect marks 1 -> 21
Other:
- moved on the sheet: J2

Commit message: quick save
Connections:
- net CHARGER_CC2: now also J1.50 (Pin_50); no longer J1.51 (Pin_51)
- net CHARGER_D+: now also J1.48 (Pin_48); no longer J1.49 (Pin_49)
- net CHARGER_D-: now also J1.47 (Pin_47); no longer J1.48 (Pin_48)
- net CHARGER_VBUS: now also J1.51 (Pin_51)
- net GNDD: now also J1.49 (Pin_49); no longer J1.47 (Pin_47), J1.50 (Pin_50)
Changed lines of the file:
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@@
-	)
-	(junction
-		(at 63.5 242.57)
-		(diameter 0)
-		(color 0 0 0 0)
 	)
 	(junction
@@
 	(wire
 		(pts
-			(xy 62.23 250.19) (xy 63.5 250.19)
-		)
-		(stroke
-			(width 0)
-			(type default)
-		)
-	)
-	(wire
-		(pts
 			(xy 38.1 146.05) (xy 48.26 146.05)
 		)
@@
 	(wire
 		(pts
-			(xy 62.23 242.57) (xy 63.5 242.57)
-		)
-		(stroke
-			(width 0)
-			(type default)
-		)
-	)
-	(wire
-		(pts
 			(xy 59.69 208.28) (xy 59.69 205.74)
 		)
@@
 	(wire
 		(pts
-			(xy 63.5 242.57) (xy 63.5 243.84)
-		)
-		(stroke
-			(width 0)
-			(type default)
-		)
-	)
-	(wire
-		(pts
 			(xy 38.1 170.18) (xy 52.07 170.18)
 		)
@@
 	(wire
 		(pts
+			(xy 50.8 241.3) (xy 63.5 241.3)
+		)
+		(stroke
+			(width 0)
+			(type default)
+		)
+	)
+	(wire
+		(pts
 			(xy 22.86 158.75) (xy 22.86 154.94)
 		)
@@
 	(wire
 		(pts
+			(xy 62.23 247.65) (xy 63.5 247.65)
+		)
+		(stroke
+			(width 0)
+			(type default)
+		)
+	)
+	(wire
+		(pts
 			(xy 54.61 147.32) (xy 63.5 147.32)
 		)
@@
 	(wire
 		(pts
+			(xy 63.5 247.65) (xy 63.5 248.92)
+		)
+		(stroke
+			(width 0)
+			(type default)
+		)
+	)
+	(wire
+		(pts
 			(xy 44.45 180.34) (xy 54.61 170.18)
 		)
@@
 	(wire
 		(pts
-			(xy 63.5 241.3) (xy 63.5 242.57)
-		)
-		(stroke
-			(width 0)
-			(type default)
-		)
-	)
-	(wire
-		(pts
 			(xy 40.64 195.58) (xy 44.45 195.58)
-		)
-		(stroke
-			(width 0)
-			(type default)
-		)
-	)
-	(wire
-		(pts
-			(xy 63.5 250.19) (xy 63.5 251.46)
 		)
 		(stroke
@@
 		)
 	)
-	(label "CHARGER_D-"
-		(at 63.5 246.38 180)
+	(label "CHARGER_VBUS"
+		(at 63.5 254 180)
 		(effects
 			(font
@@
 	)
 	(label "CHARGER_CC2"
-		(at 63.5 254 180)
-		(effects
-			(font
-				(size 1.27 1.27)
-			)
-			(justify right bottom)
-		)
-	)
-	(label "CHARGER_D+"
-		(at 63.5 248.92 180)
+		(at 63.5 251.46 180)
 		(effects
 			(font
@@
 		)
 	)
+	(label "CHARGER_D+"
+		(at 63.5 246.38 180)
+		(effects
+			(font
+				(size 1.27 1.27)
+			)
+			(justify right bottom)
+		)
+	)
 	(label "DAC_CC1"
 		(at 114.3 266.7 0)
@@
 	(label "CHARGER_VBUS"
 		(at 63.5 256.54 180)
+		(effects
+			(font
+				(size 1.27 1.27)
+			)
+			(justify right bottom)
+		)
+	)
+	(label "CHARGER_D-"
+		(at 63.5 243.84 180)
 		(effects
 			(font
@@
 	(symbol
 		(lib_id "power:GNDD")
-		(at 62.23 242.57 270)
+		(at 50.8 241.3 270)
 		(unit 1)
 		(exclude_from_sim no)
@@
 		(fields_autoplaced yes)
 		(property "Reference" "#PWR0264"
-			(at 55.88 242.57 0)
+			(at 44.45 241.3 0)
 			(effects
 				(font
@@
 		)
 		(property "Value" "GNDD"
-			(at 58.42 242.5699 90)
+			(at 46.99 241.2999 90)
 			(effects
 				(font
@@
 		)
 		(property "Footprint" ""
-			(at 62.23 242.57 0)
+			(at 50.8 241.3 0)
 			(effects
 				(font
@@
 		)
 		(property "Datasheet" ""
-			(at 62.23 242.57 0)
+			(at 50.8 241.3 0)
 			(effects
 				(font
@@
 		)
 		(property "Description" "Power symbol creates a global label with name \"GNDD\" , digital ground"
-			(at 62.23 242.57 0)
+			(at 50.8 241.3 0)
 			(effects
 				(font
@@
 	(symbol
 		(lib_id "power:GNDD")
-		(at 62.23 250.19 270)
+		(at 62.23 247.65 270)
 		(unit 1)
 		(exclude_from_sim no)
@@
 		(fields_autoplaced yes)
 		(property "Reference" "#PWR0261"
-			(at 55.88 250.19 0)
+			(at 55.88 247.65 0)
 			(effects
 				(font
@@
 		)
 		(property "Value" "GNDD"
-			(at 58.42 250.1899 90)
+			(at 58.42 247.6499 90)
 			(effects
 				(font
@@
 		)
 		(property "Footprint" ""
-			(at 62.23 250.19 0)
+			(at 62.23 247.65 0)
 			(effects
 				(font
@@
 		)
 		(property "Datasheet" ""
-			(at 62.23 250.19 0)
+			(at 62.23 247.65 0)
 			(effects
 				(font
@@
 		)
 		(property "Description" "Power symbol creates a global label with name \"GNDD\" , digital ground"
-			(at 62.23 250.19 0)
-			(effects
-				(font
+			(at 62.23 247.65 0)
+			(effects
+				(font
