File: Display/Display.kicad_sch (KiCad schematic)
At the start: 8 parts, among them J1 Conn_01x60, J2 12402032E202A, J3 12402032E202A

Commit message: update kicad version and switch #
Parts:
- S1, S2, S3, S4, S5: value TL2285OA -> TL2230OAF140; DigiKey Part # EG1871-ND -> EG6032-ND

Commit message: update ordering numbers
Parts:
- J1: DigiKey Part # (none) -> 900-2004850460CT-ND; JLCPCB Part # (none) -> C3168514
- J2, J3: DigiKey Part # (none) -> 664-12402032E202ACT-ND; JLCPCB Part # (none) -> C3198011
Changed lines of the file:
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@@
+			)
+		)
+		(property "DigiKey Part #" "664-12402032E202ACT-ND"
+			(at 114.3 276.86 0)
+			(hide yes)
+			(show_name no)
+			(do_not_autoplace no)
+			(effects
+				(font
+					(size 1.27 1.27)
+				)
+			)
+		)
+		(property "JLCPCB Part #" "C3198011"
+			(at 114.3 276.86 0)
+			(hide yes)
+			(show_name no)
+			(do_not_autoplace no)
+			(effects
+				(font
+					(size 1.27 1.27)
+				)
 			)
 		)
@@
 			)
 		)
+		(property "DigiKey Part #" "664-12402032E202ACT-ND"
+			(at 114.3 187.96 0)
+			(hide yes)
+			(show_name no)
+			(do_not_autoplace no)
+			(effects
+				(font
+					(size 1.27 1.27)
+				)
+			)
+		)
+		(property "JLCPCB Part #" "C3198011"
+			(at 114.3 187.96 0)
+			(hide yes)
+			(show_name no)
+			(do_not_autoplace no)
+			(effects
+				(font
+					(size 1.27 1.27)
+				)
+			)
+		)
 		(pin "A12"
 		)
@@
 			(at 68.58 200.66 0)
 			(hide yes)
+			(show_name no)
+			(do_not_autoplace no)
+			(effects
+				(font
+					(size 1.27 1.27)
+				)
+			)
+		)
+		(property "DigiKey Part #" "900-2004850460CT-ND"
+			(at 68.58 200.66 0)
+			(hide yes)
+			(show_name no)
+			(do_not_autoplace no)
+			(effects
+				(font
+					(size 1.27 1.27)
+				)
+			)
+		)
+		(property "JLCPCB Part #" "C3168514"
+			(at 68.58 200.66 0)
+			(hide yes)
