File: Display/Digit.kicad_sch (KiCad schematic)
At the start: 20 parts, among them U1 74HC595, U2 74HC595

Commit message: quick save
Connections:
- net c: now also U1.15 (QA); no longer U2.4 (QE)
- net d: now also U2.6 (QG); no longer U1.15 (QA)
- net e: now also U2.5 (QF); no longer U2.6 (QG)
- net p: now also U2.4 (QE); no longer U2.5 (QF)
Changed lines of the file:
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@@
 	)
 	(label "p"
-		(at 153.67 125.73 0)
+		(at 153.67 123.19 0)
 		(effects
 			(font
@@
 	)
 	(label "d"
-		(at 153.67 68.58 0)
+		(at 153.67 128.27 0)
 		(effects
 			(font
@@
 	)
 	(label "c"
-		(at 153.67 123.19 0)
+		(at 153.67 68.58 0)
 		(effects
 			(font
@@
 	)
 	(label "e"
-		(at 153.67 128.27 0)
-		(effects
-			(font
+		(at 153.67 125.73 0)
+		(effects
+			(font

Commit message: add C Part #
Parts:
- C1, C2: LCSC (none) -> C49062
Changed lines of the file:
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@@
+			)
+		)
+		(property "LCSC" "C49062"
+			(at 113.03 135.89 0)
+			(effects
+				(font
+					(size 1.27 1.27)
+				)
+				(hide yes)
 			)
 		)
@@
 			(at 97.79 135.89 0)
 			(effects
+				(font
+					(size 1.27 1.27)
+				)
+				(hide yes)
+			)
+		)
+		(property "LCSC" "C49062"
+			(at 97.79 135.89 0)
+			(effects
