File: Display/Digit.kicad_sch (KiCad schematic)
At the start: 20 parts, among them U1 74HC595, U2 74HC595

Commit message: update kicad version and switch #
Parts:
- SEGD1: value ~ -> (none)

Commit message: update ordering numbers
Parts:
- C1, C2: JLCPCB Part # (none) -> C49062; LCSC C49062 -> (none)
- R1, R10, R11, R12, R13, R14, R15, R2, R3, R4, R5, R6, R7, R8, R9: JLCPCB Part # (none) -> C25076; LCSC C25076 -> (none)
- SEGD1: DigiKey ACPSC04-41SEKWA -> (none); DigiKey Part # (none) -> 754-ACPSC04-41SEKWACT-ND; JLCPCB Part # (none) -> C6854600
- U1: DigiKey 74HC595PW,118 -> (none); DigiKey Part # (none) -> 1727-3068-1-ND; JLCPCB Part # (none) -> C5948
- U2: DigiKey Part # (none) -> 1727-3068-1-ND; JLCPCB Part # (none) -> C5948
Changed lines of the file:
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@@
 			)
 		)
-		(property "DigiKey" "ACPSC04-41SEKWA"
+		(property "DigiKey Part #" "754-ACPSC04-41SEKWACT-ND"
+			(at 198.12 77.47 0)
+			(hide yes)
+			(show_name no)
+			(do_not_autoplace no)
+			(effects
+				(font
+					(size 1.27 1.27)
+				)
+			)
+		)
+		(property "JLCPCB Part #" "C6854600"
 			(at 198.12 77.47 0)
 			(hide yes)
@@
 			)
 		)
-		(property "LCSC" "C25076"
+		(property "JLCPCB Part #" "C25076"
 			(at 182.88 78.74 90)
 			(hide yes)
@@
 			)
 		)
-		(property "LCSC" "C25076"
+		(property "JLCPCB Part #" "C25076"
 			(at 182.88 115.57 90)
 			(hide yes)
@@
 			)
 		)
-		(property "LCSC" "C25076"
+		(property "JLCPCB Part #" "C25076"
 			(at 182.88 83.82 90)
 			(hide yes)
@@
 			)
 		)
-		(property "LCSC" "C25076"
+		(property "JLCPCB Part #" "C25076"
 			(at 182.88 118.11 90)
 			(hide yes)
@@
 			)
 		)
-		(property "LCSC" "C25076"
+		(property "JLCPCB Part #" "C25076"
 			(at 182.88 123.19 90)
 			(hide yes)
@@
 			)
 		)
-		(property "LCSC" "C25076"
+		(property "JLCPCB Part #" "C25076"
 			(at 182.88 76.2 90)
 			(hide yes)
@@
 			)
 		)
-		(property "DigiKey" "74HC595PW,118"
+		(property "DigiKey Part #" "1727-3068-1-ND"
+			(at 143.51 78.74 0)
+			(hide yes)
+			(show_name no)
+			(do_not_autoplace no)
+			(effects
+				(font
+					(size 1.27 1.27)
+				)
+			)
+		)
+		(property "JLCPCB Part #" "C5948"
 			(at 143.51 78.74 0)
 			(hide yes)
@@
 			)
 		)
-		(property "LCSC" "C25076"
+		(property "JLCPCB Part #" "C25076"
 			(at 182.88 125.73 90)
 			(hide yes)
@@
 			)
 		)
-		(property "LCSC" "C25076"
+		(property "JLCPCB Part #" "C25076"
 			(at 182.88 113.03 90)
 			(hide yes)
@@
 			)
 		)
-		(property "LCSC" "C25076"
+		(property "JLCPCB Part #" "C25076"
 			(at 182.88 71.12 90)
 			(hide yes)
@@
 			)
 		)
+		(property "DigiKey Part #" "1727-3068-1-ND"
+			(at 143.51 123.19 0)
+			(hide yes)
+			(show_name no)
+			(do_not_autoplace no)
+			(effects
+				(font
+					(size 1.27 1.27)
+				)
+			)
+		)
+		(property "JLCPCB Part #" "C5948"
+			(at 143.51 123.19 0)
+			(hide yes)
+			(show_name no)
+			(do_not_autoplace no)
+			(effects
+				(font
+					(size 1.27 1.27)
+				)
+			)
+		)
 		(pin "13"
 		)
@@
 			)
 		)
-		(property "LCSC" "C25076"
+		(property "JLCPCB Part #" "C25076"
 			(at 182.88 81.28 90)
 			(hide yes)
@@
 			)
 		)
-		(property "LCSC" "C25076"
+		(property "JLCPCB Part #" "C25076"
 			(at 182.88 120.65 90)
 			(hide yes)
@@
 			)
 		)
-		(property "LCSC" "C49062"
+		(property "JLCPCB Part #" "C49062"
 			(at 113.03 135.89 0)
 			(hide yes)
@@
 			)
 		)
-		(property "LCSC" "C25076"
+		(property "JLCPCB Part #" "C25076"
 			(at 182.88 68.58 90)
 			(hide yes)
@@
 			)
 		)
-		(property "LCSC" "C49062"
+		(property "JLCPCB Part #" "C49062"
 			(at 97.79 135.89 0)
 			(hide yes)
@@
 			)
 		)
-		(property "LCSC" "C25076"
+		(property "JLCPCB Part #" "C25076"
 			(at 182.88 73.66 90)
 			(hide yes)
@@
 			)
 		)
-		(property "LCSC" "C25076"
+		(property "JLCPCB Part #" "C25076"
 			(at 182.88 128.27 90)
 			(hide yes)
@@
 			)
 		)
-		(property "LCSC" "C25076"
+		(property "JLCPCB Part #" "C25076"
 			(at 182.88 86.36 90)
 			(hide yes)

Commit message: Update Digit.kicad_sch
Parts:
- C1, C2: DigiKey Part # (none) -> 1276-1115-1-ND
- R1, R10, R11, R12, R13, R14, R15, R2, R3, R4, R5, R6, R7, R8, R9: DigiKey Part # (none) -> 311-100LRCT-ND
Changed lines of the file:
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@@
 			)
 		)
+		(property "DigiKey Part #" "311-100LRCT-ND"
+			(at 182.88 78.74 90)
+			(hide yes)
+			(show_name no)
+			(do_not_autoplace no)
+			(effects
+				(font
+					(size 1.27 1.27)
+				)
+			)
+		)
 		(pin "2"
 		)
@@
 			)
 		)
+		(property "DigiKey Part #" "311-100LRCT-ND"
+			(at 182.88 115.57 90)
+			(hide yes)
+			(show_name no)
+			(do_not_autoplace no)
+			(effects
+				(font
+					(size 1.27 1.27)
+				)
+			)
+		)
 		(pin "2"
 		)
@@
 			)
 		)
+		(property "DigiKey Part #" "311-100LRCT-ND"
+			(at 182.88 83.82 90)
+			(hide yes)
+			(show_name no)
+			(do_not_autoplace no)
+			(effects
+				(font
+					(size 1.27 1.27)
+				)
+			)
+		)
 		(pin "2"
 		)
@@
 			)
 		)
+		(property "DigiKey Part #" "311-100LRCT-ND"
+			(at 182.88 118.11 90)
+			(hide yes)
+			(show_name no)
+			(do_not_autoplace no)
+			(effects
+				(font
+					(size 1.27 1.27)
+				)
+			)
+		)
 		(pin "2"
 		)
@@
 			)
 		)
+		(property "DigiKey Part #" "311-100LRCT-ND"
+			(at 182.88 123.19 90)
+			(hide yes)
+			(show_name no)
+			(do_not_autoplace no)
+			(effects
+				(font
+					(size 1.27 1.27)
+				)
+			)
+		)
 		(pin "2"
 		)
@@
 			)
 		)
+		(property "DigiKey Part #" "311-100LRCT-ND"
+			(at 182.88 76.2 90)
+			(hide yes)
+			(show_name no)
+			(do_not_autoplace no)
+			(effects
+				(font
+					(size 1.27 1.27)
+				)
+			)
+		)
 		(pin "2"
 		)
@@
 			)
 		)
+		(property "DigiKey Part #" "311-100LRCT-ND"
+			(at 182.88 125.73 90)
+			(hide yes)
+			(show_name no)
+			(do_not_autoplace no)
+			(effects
+				(font
+					(size 1.27 1.27)
+				)
+			)
+		)
 		(pin "2"
 		)
@@
 			)
 		)
+		(property "DigiKey Part #" "311-100LRCT-ND"
+			(at 182.88 113.03 90)
+			(hide yes)
+			(show_name no)
+			(do_not_autoplace no)
+			(effects
+				(font
+					(size 1.27 1.27)
+				)
+			)
+		)
 		(pin "2"
 		)
@@
 			)
 		)
+		(property "DigiKey Part #" "311-100LRCT-ND"
+			(at 182.88 71.12 90)
+			(hide yes)
+			(show_name no)
+			(do_not_autoplace no)
+			(effects
+				(font
+					(size 1.27 1.27)
+				)
+			)
+		)
 		(pin "2"
 		)
@@
 			)
 		)
+		(property "DigiKey Part #" "311-100LRCT-ND"
+			(at 182.88 81.28 90)
+			(hide yes)
+			(show_name no)
+			(do_not_autoplace no)
+			(effects
+				(font
+					(size 1.27 1.27)
+				)
+			)
+		)
 		(pin "2"
 		)
@@
 			)
 		)
+		(property "DigiKey Part #" "311-100LRCT-ND"
+			(at 182.88 120.65 90)
+			(hide yes)
+			(show_name no)
+			(do_not_autoplace no)
+			(effects
+				(font
+					(size 1.27 1.27)
+				)
+			)
+		)
 		(pin "2"
 		)
@@
 			)
 		)
+		(property "DigiKey Part #" "1276-1115-1-ND"
+			(at 113.03 135.89 0)
+			(hide yes)
+			(show_name no)
+			(do_not_autoplace no)
+			(effects
+				(font
+					(size 1.27 1.27)
+				)
+			)
+		)
 		(pin "1"
 		)
@@
 			)
 		)
+		(property "DigiKey Part #" "311-100LRCT-ND"
+			(at 182.88 68.58 90)
+			(hide yes)
+			(show_name no)
+			(do_not_autoplace no)
+			(effects
+				(font
+					(size 1.27 1.27)
+				)
+			)
+		)
 		(pin "2"
 		)
@@
 			)
 		)
+		(property "DigiKey Part #" "1276-1115-1-ND"
+			(at 97.79 135.89 0)
+			(hide yes)
+			(show_name no)
+			(do_not_autoplace no)
+			(effects
+				(font
+					(size 1.27 1.27)
+				)
+			)
+		)
 		(pin "1"
 		)
@@
 			)
 		)
+		(property "DigiKey Part #" "311-100LRCT-ND"
+			(at 182.88 73.66 90)
+			(hide yes)
+			(show_name no)
+			(do_not_autoplace no)
+			(effects
+				(font
+					(size 1.27 1.27)
+				)
+			)
+		)
 		(pin "2"
 		)
@@
 			)
 		)
+		(property "DigiKey Part #" "311-100LRCT-ND"
+			(at 182.88 128.27 90)
+			(hide yes)
+			(show_name no)
+			(do_not_autoplace no)
+			(effects
+				(font
+					(size 1.27 1.27)
+				)
+			)
+		)
 		(pin "2"
 		)
@@
 			(at 182.88 86.36 90)
 			(hide yes)
+			(show_name no)
+			(do_not_autoplace no)
+			(effects
+				(font
+					(size 1.27 1.27)
+				)
+			)
+		)
+		(property "DigiKey Part #" "311-100LRCT-ND"
+			(at 182.88 86.36 90)
+			(hide yes)
