File: Display/Display.kicad_pcb (KiCad board)
At the start: 4 copper layers, 177.2 x 47 mm, 573 parts, among them J1 Conn_01x60, J2 12402032E202A, J3 12402032E202A, U1 74HC595, U10 74HC595, U11 74HC595, U12 74HC595, U13 74HC595, U14 74HC595, U15 74HC595, U16 74HC595, U17 74HC595, U18 74HC595, U19 74HC595, U2 74HC595, U20 74HC595, U21 74HC595, U22 74HC595, U23 74HC595, U24 74HC595, U25 74HC595, U26 74HC595, U27 74HC595, U28 74HC595, U29 74HC595, U3 74HC595, U30 74HC595, U31 74HC595, U32 74HC595, U33 74HC595, U34 74HC595, U35 74HC595, U36 74HC595, U37 74HC595, U38 74HC595, U39 74HC595, U4 74HC595, U40 74HC595, U41 74HC595, U42 74HC595, U43 74HC595, U44 74HC595, U45 74HC595, U46 74HC595, U47 74HC595, U48 74HC595, U49 74HC595, U5 74HC595, U50 74HC595, U51 74HC595, U52 74HC595, U53 74HC595, U54 74HC595, U55 74HC595, U56 74HC595, U6 74HC595, U7 74HC595, U8 74HC595, U9 74HC595

Commit message: update kicad version and switch #
Parts:
- S1, S2, S3, S4, S5: value TL2285OA -> TL2230OAF140
