File: Amplifier/Amplifier.kicad_sch (KiCad schematic)
At the start: 7 parts, among them J108 Prog BT, U103 ESP32-WROOM-32U

Commit message: user save
Parts:
- added J1: Conn_01x60, External_Parts:CON_2004850460_MOL, symbol Connector_Generic:Conn_01x60
- added R3, R4: 10k, Resistor_THT:R_Axial_DIN0207_L6.3mm_D2.5mm_P10.16mm_Horizontal, symbol Device:R
- added R5, R6: 0R, Resistor_THT:R_Axial_DIN0207_L6.3mm_D2.5mm_P10.16mm_Horizontal, symbol Device:R
- added S1, S2, S3, S4, S5: TL2230EEF100, External_Parts:SW_TL2230EEF100, symbol External_Parts:TL2230EEF100
- U103: DigiKey Part # (none) -> ESP32-WROOM-32E-N16
Connections:
- new net: J1.51 (Pin_51), R5.1
- new net: J1.29 (Pin_29), S5.1
- new net: J1.27 (Pin_27), S5.2
- new net: J1.25 (Pin_25), S5.3
- new net: J1.30 (Pin_30), S5.4
- new net: J1.28 (Pin_28), S5.5
- new net: J1.26 (Pin_26), S5.6
- new net: J1.11 (Pin_11), S2.1
- new net: J1.9 (Pin_9), S2.2
- new net: J1.7 (Pin_7), S2.3
- new net: J1.12 (Pin_12), S2.4
- new net: J1.10 (Pin_10), S2.5
- new net: J1.8 (Pin_8), S2.6
- new net: J1.13 (Pin_13), S3.1
- new net: J1.15 (Pin_15), S3.2
- new net: J1.17 (Pin_17), S3.3
- new net: J1.14 (Pin_14), S3.4
- new net: J1.16 (Pin_16), S3.5
- new net: J1.18 (Pin_18), S3.6
- new net: J1.52 (Pin_52), R6.1
- new net: J1.1 (Pin_1), S1.1
- new net: J1.3 (Pin_3), S1.2
- new net: J1.5 (Pin_5), S1.3
- new net: J1.2 (Pin_2), S1.4
- new net: J1.4 (Pin_4), S1.5
- new net: J1.6 (Pin_6), S1.6
- new net: J1.23 (Pin_23), S4.1
- new net: J1.21 (Pin_21), S4.2
- new net: J1.19 (Pin_19), S4.3
- new net: J1.24 (Pin_24), S4.4
- new net: J1.22 (Pin_22), S4.5
- new net: J1.20 (Pin_20), S4.6
- new net: J1.53 (Pin_53), R4.1
- new net: J1.50 (Pin_50), R3.1
- new net +5V: R3.2, R4.2
- new net CHARGER_VBUS: R5.2, R6.2
- new net DAC_CC1: J1.60 (Pin_60)
- new net DAC_CC2: J1.54 (Pin_54)
- new net DAC_D+: J1.56 (Pin_56)
- new net DAC_D-: J1.57 (Pin_57)
- new net DAC_VBUS: J1.59 (Pin_59)
- new net GNDD: J1.36 (Pin_36), J1.38 (Pin_38), J1.40 (Pin_40), J1.42 (Pin_42), J1.44 (Pin_44), J1.46 (Pin_46), J1.49 (Pin_49), J1.55 (Pin_55), J1.58 (Pin_58)
- new net RCL: J1.41 (Pin_41)
- new net SR: J1.37 (Pin_37)
- new net SRCL: J1.43 (Pin_43)
- new net SRCR: J1.45 (Pin_45)
- new net VCC: J1.31 (Pin_31), J1.32 (Pin_32), J1.33 (Pin_33), J1.34 (Pin_34), J1.35 (Pin_35)
- new net ~{OE}: J1.39 (Pin_39)
- no-connect marks 18 -> 20
