File: DAC_EVT/DAC_EVT.kicad_sch (KiCad schematic)
At the start: 0 parts

Commit message: production
Parts:
- added C101, C106, C109, C111, C113, C114, C115, C116: 0u1, Capacitor_SMD:C_0402_1005Metric_Pad0.74x0.62mm_HandSolder, symbol Device:C
- added C102, C103: 2n2, Capacitor_SMD:C_0402_1005Metric_Pad0.74x0.62mm_HandSolder, symbol Device:C
- added C104, C107: 2u2, Capacitor_THT:CP_Radial_D5.0mm_P2.00mm, symbol Device:C_Polarized
- added C105, C108, C110, C112: 10u, Capacitor_THT:CP_Radial_D5.0mm_P2.00mm, symbol Device:C_Polarized
- added J101: Conn_02x20_Odd_Even, Connector_PinHeader_2.54mm:PinHeader_2x20_P2.54mm_Vertical, symbol Connector_Generic:Conn_02x20_Odd_Even
- added J102: SJ1-3523N, external_components:CUI_SJ1-3523N, symbol external_components:SJ1-3523N
- added J103: Conn_01x04_Socket, Connector_PinSocket_2.54mm:PinSocket_1x04_P2.54mm_Vertical, symbol Connector:Conn_01x04_Socket
- added J104, J105: Conn_01x03_Socket, Connector_PinSocket_2.54mm:PinSocket_1x03_P2.54mm_Vertical, symbol Connector:Conn_01x03_Socket
- added J106: Screw_Terminal_01x02, TerminalBlock_Phoenix:TerminalBlock_Phoenix_MKDS-1,5-2_1x02_P5.00mm_Horizontal, symbol Connector:Screw_Terminal_01x02
- added J107, J108: Conn_01x20_Pin, Connector_PinHeader_2.54mm:PinHeader_1x20_P2.54mm_Vertical, symbol Connector:Conn_01x20_Pin
- added R101, R102, R103, R104, R105: 470, Resistor_SMD:R_0603_1608Metric_Pad0.98x0.95mm_HandSolder, symbol Device:R
- added U101: PCM5102A, Package_SO:TSSOP-20_4.4x6.5mm_P0.65mm, symbol Audio:PCM5102A
- added U102: NE5532, Package_SO:SOIC-8_3.9x4.9mm_P1.27mm, symbol Amplifier_Operational:NE5532
- added U103: TCR2EF33_LMCT, external_components:SOT-25 SMV_TOS, symbol external_components:TCR2EF33_LMCT
Connections:
- new net: C107.1, U101.5 (VNEG)
- new net: C104.1, U101.2 (CAPP)
- new net: C104.2, U101.4 (CAPM)
- new net: R101.1, U101.7 (OUTR)
- new net: C102.2, R101.2, U102.5 (+)
- new net: R104.1, U102.6 (-)
- new net: J102.3, R104.2, U102.7
- new net: J102.2, R103.2, U102.1
- new net: R103.1, U102.2 (-)
- new net: C103.2, R102.2, U102.3 (+)
- new net: J101.1 (Pin_1), J107.1 (Pin_1)
- new net: J101.19 (Pin_19), J107.10 (Pin_10)
- new net: J101.21 (Pin_21), J107.11 (Pin_11)
- new net: J101.23 (Pin_23), J107.12 (Pin_12)
- new net: J101.25 (Pin_25), J107.13 (Pin_13)
- new net: J101.27 (Pin_27), J107.14 (Pin_14)
- new net: J101.29 (Pin_29), J107.15 (Pin_15)
- new net: J101.31 (Pin_31), J107.16 (Pin_16)
- new net: J101.33 (Pin_33), J107.17 (Pin_17)
- new net: J101.37 (Pin_37), J107.19 (Pin_19)
- new net: J101.3 (Pin_3), J107.2 (Pin_2)
- new net: J101.39 (Pin_39), J107.20 (Pin_20)
- new net: J101.5 (Pin_5), J107.3 (Pin_3)
- new net: J101.7 (Pin_7), J107.4 (Pin_4)
- new net: J101.9 (Pin_9), J107.5 (Pin_5)
- new net: J101.11 (Pin_11), J107.6 (Pin_6)
- new net: J101.13 (Pin_13), J107.7 (Pin_7)
- new net: J101.15 (Pin_15), J107.8 (Pin_8)
- new net: J101.17 (Pin_17), J107.9 (Pin_9)
- new net: J103.1 (Pin_1), R105.1
- new net: C105.1, C106.2, U101.18 (LDOO)
- new net: C114.2, J103.4 (Pin_4), U102.8 (V+)
- new net: R102.1, U101.6 (OUTL)
- new net: J101.2 (Pin_2), J108.1 (Pin_1)
- new net: J101.20 (Pin_20), J108.10 (Pin_10)
- new net: J101.22 (Pin_22), J108.11 (Pin_11)
- new net: J101.24 (Pin_24), J108.12 (Pin_12)
- new net: J101.26 (Pin_26), J108.13 (Pin_13)
- new net: J101.28 (Pin_28), J108.14 (Pin_14)
- new net: J101.30 (Pin_30), J108.15 (Pin_15)
- new net: J101.32 (Pin_32), J108.16 (Pin_16)
- new net: J101.34 (Pin_34), J108.17 (Pin_17)
- new net: J101.36 (Pin_36), J108.18 (Pin_18)
- new net: J101.38 (Pin_38), J108.19 (Pin_19)
- new net: J101.8 (Pin_8), J108.4 (Pin_4)
- new net: J101.10 (Pin_10), J108.5 (Pin_5)
- new net: J101.14 (Pin_14), J108.7 (Pin_7)
- new net: J101.16 (Pin_16), J108.8 (Pin_8)
- new net: J101.18 (Pin_18), J108.9 (Pin_9)
- new net: C113.2, J103.3 (Pin_3), U102.4 (V-)
- new net +5V: C116.2, J101.4 (Pin_4), J104.3 (Pin_3), J106.1 (Pin_1), J108.2 (Pin_2), R105.2, U103.1 (VIN), U103.3 (CONTROL)
- new net GND: C101.1, C102.1, C103.1, C105.2, C106.1, C107.2, C108.2, C109.1, C110.2, C111.1, C112.2, C113.1, C114.1, C115.1, C116.1, J101.6 (Pin_6), J102.1, J103.2 (Pin_2), J104.1 (Pin_1), J105.1 (Pin_1), J105.2 (Pin_2), J105.3 (Pin_3), J106.2 (Pin_2), J108.3 (Pin_3), U101.10 (DEMP), U101.11 (FLT), U101.12 (SCK), U101.16 (FMT), U101.19 (DGND), U101.3 (CPGND), U101.9 (AGND), U103.2 (GND)
- new net I2S_BCLK: J101.12 (Pin_12), J108.6 (Pin_6), U101.13 (BCK)
- new net I2S_LRCLK: J101.35 (Pin_35), J107.18 (Pin_18), U101.15 (LRCK)
- new net I2S_SDATA: J101.40 (Pin_40), J108.20 (Pin_20), U101.14 (DIN)
- new net ~{DAC_Mute}: C101.2, C108.1, C109.2, C110.1, C111.2, C112.1, C115.2, U101.1 (CPVDD), U101.17 (XSMT), U101.20 (DVDD), U101.8 (AVDD), U103.5 (VOUT)
- no-connect marks 0 -> 1
Changed lines of the file:
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@@
 	(generator_version "9.0")
 	(paper "A4")
-	(sheet_instances
-		(path "/"
-			(page "1")
-		)
-	)
-	(embedded_fonts no)
-)
