File: Systemboard/Systemboard.kicad_sch (KiCad schematic)
At the start: 23 parts, among them J1 Conn_01x60, J108 Prog BT, J2 Conn_01x02, J3 Conn_01x01, J4 Conn_01x01, U101 ESP32-WROOM-32E

Commit message: Update Systemboard.kicad_sch
Parts:
- J1: JLCPCB Part # (none) -> C3168514
Changed lines of the file:
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@@
 			)
 		)
-		(property "JLCPCB Part #" ""
+		(property "JLCPCB Part #" "C3168514"
 			(at 31.75 102.87 0)
 			(hide yes)
