File: Systemboard/Systemboard.kicad_pcb (KiCad board)
At the start: 4 copper layers, 175 x 135 mm, 208 parts, among them J1 Conn_01x60, J108 Prog BT, J2 Conn_01x02, J3 Conn_01x01, J4 Conn_01x01, Q1 MMBT5551L, Q2 MMBT5551L, Q3 MMBT5551L, Q4 MMBT5551L, Q5 MMBT5551L, U1 INA226, U10 74HC595, U101 ESP32-WROOM-32E, U103 TLV73333PDBV, U104 PCM2706CPJTR, U11 74HC14, U2 LM358, U201 TLV73333PDBV, U202 PCM5102A, U3 J104D2C12VDC.15S, U301 TLV73333PDBV, U4 J104D2C12VDC.15S, U5 LM2596S-5, U501 TPA3118D2DAPR, U6 LM2596S-3.3, U7 LM2596S-5, U8 LM2596S-ADJ, U9 LTV-817S, Y101 CSTNE12M0G55A000R0

Commit message: B+ width adjusted
Routing:
- net /+B: track 35.8 -> 28.8 mm
Changed lines of the file:
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@@
-	)
-	(segment
-		(start 165.6187 46.3133)
-		(end 165.6187 42.5036)
-		(width 0.2)
-		(layer "B.Cu")
-		(net "/+B")
 	)
 	(segment
 		(start 171.835 36.287)
 		(end 171.835 33.1783)
-		(width 0.4)
+		(width 1)
 		(layer "B.Cu")
 		(net "/+B")
@@
 		(start 165.619 46.3136)
 		(end 165.619 42.5036)
-		(width 0.4)
-		(layer "B.Cu")
-		(net "/+B")
-	)
-	(segment
-		(start 171.8353 33.178)
-		(end 171.8353 30.0696)
-		(width 0.2)
+		(width 1)
 		(layer "B.Cu")
 		(net "/+B")
@@
 		(start 165.619 42.5036)
 		(end 171.835 36.287)
-		(width 0.4)
+		(width 1)
 		(layer "B.Cu")
 		(net "/+B")
@@
 		(start 171.835 33.1783)
 		(end 171.835 30.0696)
-		(width 0.4)
+		(width 1)
 		(layer "B.Cu")
 		(net "/+B")
@@
 		(start 165.619 50.1236)
 		(end 165.619 46.3136)
-		(width 0.4)
+		(width 1)
 		(layer "B.Cu")
 		(net "/+B")

Commit message: fix amp pullup value
was too high. amp was not turning on
Parts:
- R504: value 100k -> 47k
Changed lines of the file:
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@@
 			(unit
 				(name "A")
-				(pins "3" "4" "5" "21" "22" "17" "18" "20" "19" "32" "2" "1" "38" "15"
-					"39" "25" "35" "24" "34" "26" "29" "14" "16" "13" "23" "27" "28" "30"
+				(pins "3" "4" "5" "21" "22" "17" "18" "20" "19" "32" "2" "1" "38" "39"
+					"15" "25" "35" "24" "34" "26" "29" "14" "16" "13" "23" "27" "28" "30"
 					"31" "33" "36" "37" "10" "11" "12" "8" "9" "6" "7"
 				)
@@
 			)
 		)
-		(property "Value" "100k"
+		(property "Value" "47k"
 			(at 0 1.43 90)
 			(layer "F.Fab")
@@
 			(keep_text_aligned yes)
 		)
-		(gr_text "3.5"
+		(gr_text "3,5"
 			(at 31.85 153.25 90)
 			(layer "F.Fab")
@@
 			(keep_text_aligned yes)
 		)
-		(gr_text "8.5"
+		(gr_text "8,5"
 			(at 28.85 155.75 90)
 			(layer "F.Fab")
